Commit message: adding the ekf localization and adjusting the controllers to work with rotaions

File: bluerov2_description/urdf/bluerov2_alpha/bluerov2_alpha.xacro (robot description, xacro)
@@ -8,5 +8,5 @@
   <xacro:arg name="initial_positions_file" default="initial_positions.yaml" />
   <xacro:arg name="namespace" default="bluerov/" />
-  <xacro:arg name="prefix" default="bluerov/" />
+  <xacro:arg name="prefix" default="" />
   <xacro:arg name="use_sim" default="true" />
   <xacro:arg name="description_package" default="bluerov2_cirtesu_core" />

File: bluerov2_description/urdf/cirtesu/cirtesu.urdf.xacro (robot description, xacro)
@@ -3,8 +3,5 @@
   <!-- Define a material with a texture -->
   <material name="cirtesu_material">
-    <texture filename="$(find bluerov2_cirtesu_core)/resources/cirtesu/tank_tex.png"/>
-  </material>
-  <material name="poster_material">
-    <texture filename="$(find bluerov2_cirtesu_core)/resources/cirtesu/poster_pool_small_tex.png"/>
+    <texture filename="$(find bluerov2_description)/resources/cirtesu/tank_tex.png"/>
   </material>
   <!-- Define the base link with visual and collision elements -->
@@ -14,25 +11,8 @@
       <origin xyz="0 0 0" rpy="0 0 0"/>
       <geometry>
-        <mesh filename="package://bluerov2_cirtesu_core/resources/cirtesu/cirtesu.dae" scale="1 1 1"/>
+        <mesh filename="package://bluerov2_description/resources/cirtesu/cirtesu.dae" scale="1 1 1"/>
       </geometry>
-      <material name="poster_material"/>
+      <material name="cirtesu_material"/>
     </visual>
   </link>
   </robot>
-  <!-- Define the rectangular link with visual element -->
-  <!-- <link name="poster_link">
-    <visual>
-      <origin xyz="0 0 0.2" rpy="0 0 0"/>
-      <geometry>
-        <box size="3.5 -7.5 0.1"/>
-      </geometry>
-      <material name="poster_material"/>
-    </visual>
-  </link> -->
-  <!-- Define a joint to connect the rectangular link to the base link -->
-  <!-- <joint name="poster_joint" type="fixed">
-    <parent link="cirtesu_tank"/>
-    <child link="poster_link"/>
-    <origin xyz="0 0 -5" rpy="0 0 1.5708"/>
-  </joint>
- -->
